File: A2Pico.v2.6/A2Pico.v2.6.kicad_pcb (KiCad board)
At the start: 2 copper layers, 65.5 x 69.4 mm, 87 parts, among them J1 PinHeader_1x03_P2.54mm_Vertic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, J2 PinHeader_1x04_P2.54mm_Horizo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, T1 TO-92L_Inline_Wide, U1 Pico / PicoW, U2 74LVC245, U3 74LVC245, U4 74LVC245, U5 74F11

Commit message: Add files via upload
Parts:
- moved T1 5.08 mm to (163.8, 109.2), turned to 180 degrees
Connections:
- T1 pad 1: IRQ -> GND
- T1 pad 3: GND -> IRQ
