File: A2Pico.v2.6/A2Pico.v2.6.kicad_sch (KiCad schematic)
At the start: 27 parts, among them J1 Slide_Sw, J2 Conn_01x04, J3 Micro_SD_Card, J4 Apple2_slot, T1 BS170, U1 RPI-Pico, U2 74LVC245, U3 74LVC245, U4 74LVC245, U5 74F11

Commit message: Add files via upload
Parts:
- removed T1: BS170, Package_TO_SOT_THT:TO-92_Inline, symbol Transistor_FET:BS170
- added T1: 2N7002, Package_TO_SOT_SMD:SOT-23, symbol Transistor_FET:2N7002
Connections:
- net GND: now also T1.2 (S)
- net at J4.30 (~{IRQ}): now also T1.3 (D)
- net at R17.1, R17.2: now also T1.1 (G)
